File: Electrical/Hardware/Schematics/QORVO_RADIO2.kicad_pcb (KiCad board)
At the start: 6 copper layers, 63.5 x 63.5 mm, 61 parts, among them IC3 ADS1114BQDGSRQ1, J3 22032041, J4 22032021, J5 22032041, SW1 OS102011MS2QN1, U10 22032021, U16 LDO40LPU33RY, U17 LDO40LPU33RY, Y1 8Q-32.000MEEV-T

Commit message: Add files via upload
Parts:
- added J1: GRPB052VWQS-RC, GRPB052VWQS-RC:CONN_GRPB052_SUL, F.Cu at (154.7, 78.0)
- R1: value ERJ-3RQF1R0V -> CRCW08051R00FKEAHP; footprint Resistor_SMD:R_0603_1608Metric -> Resistor_SMD:R_0805_2012Metric
- moved L3 4.33 mm to (147.8, 98.0)
- moved R1 3.36 mm to (140.6, 77.6), turned to 0 degrees
- moved C19 3.25 mm to (142.9, 106.4)
- moved C22 3.25 mm to (133.8, 109.3)
- moved C6 3.25 mm to (146.6, 93.4)
- moved U3 3.25 mm to (153.0, 94.5)
- moved BT1 3.25 mm to (133.7, 56.1)
- moved CR2 3.25 mm to (150.0, 64.1)
- moved BT2 3.25 mm to (133.7, 65.2)
- moved C1 3.25 mm to (162.5, 62.4)
- moved C11 3.25 mm to (173.2, 97.7)
- moved C12 3.25 mm to (171.4, 95.7)
- moved C13 3.25 mm to (164.9, 98.2)
- moved C14 3.25 mm to (163.2, 98.2)
- moved C15 3.25 mm to (170.4, 90.5)
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Connections:
- R1 pad 1: /V_Source2 -> /V_Source1
- R1 pad 2: /V_Source1 -> /V_Source2
- U16 pad 7: unconnected-(U16-EPAD-Pad7) -> GND
- U17 pad 7: unconnected-(U17-EPAD-Pad7) -> GND
Routing:
- net /JTAG_TCK: track 0.00 -> 33.6 mm, vias 0 -> 2
- net /JTAG_TMS: track 0.00 -> 29.9 mm, vias 0 -> 2
- net /JTAG_TDI: track 0.00 -> 20.9 mm, vias 0 -> 2
- net /JTAG_TDO: track 0.00 -> 20.6 mm, vias 0 -> 2
- net /JTAG_nRESET: track 0.00 -> 20.3 mm, vias 0 -> 2
- net GND: track 89.1 -> 103.2 mm, vias 17 -> 18
- net +3.3V: track 42.0 -> 44.1 mm, vias 10 -> 11
- net Net-(U3-LXL_GPIO20): track 5.53 -> 7.47 mm
- net Net-(U3-LXH_GPIO19): track 5.20 -> 7.11 mm
- net +5V: track 178.7 -> 180.1 mm, vias 0 -> 1
- net /CLOCK: track 7.18 -> 7.86 mm
- net /Data -: vias 2 -> 1
- net /Data +: vias 2 -> 1
- net /DB_GPIO: vias 2 -> 1
- added copper zone on F.Cu, net (none)
Other:
- board text added: "*"

Commit message: Add files via upload
Parts:
- moved L3 0.32 mm to (147.8, 97.7)
- moved InvertedF1 0.23 mm to (126.4, 99.0)
Routing:
- net /GNDRF1: track 3.56 -> 61.1 mm
- net /GNDRF0: track 2.10 -> 51.5 mm
- net /RF0: track 2.04 -> 28.0 mm
- net /RF1: track 2.78 -> 20.6 mm

Commit message: Add files via upload
Parts:
- removed IC3: ADS1114BQDGSRQ1, ADS1114BQDGSRQ1:SOP50P490X110-10N
- removed R11, R8, R9: RMCF0603FG1K00, Resistor_SMD:R_0603_1608Metric
- added C10: 600S180FT250XT, Capacitor_SMD:C_0603_1608Metric, F.Cu at (140.4, 97.4)
- added C29: 600S1R5BT250XT4K, Capacitor_SMD:C_0603_1608Metric, F.Cu at (142.8, 100.6)
- added C3: CL10B104JB8NNNC, Capacitor_SMD:C_0603_1608Metric, F.Cu at (173.3, 102.0)
- added C30: 600S1R5BT250XT4K, Capacitor_SMD:C_0603_1608Metric, F.Cu at (142.8, 88.7)
- added C31: 600S2R2AT250XT4K, Capacitor_SMD:C_0603_1608Metric, F.Cu at (140.5, 90.0)
- added C32: 600S2R2AT250XT4K, Capacitor_SMD:C_0603_1608Metric, F.Cu at (140.4, 102.0)
- added C4: CL10A106KP8NNNC, Capacitor_SMD:C_0603_1608Metric, F.Cu at (173.3, 103.6)
- added C7: 600S180FT250XT, Capacitor_SMD:C_0603_1608Metric, F.Cu at (140.4, 81.9)
- added C8: 600S180FT250XT, Capacitor_SMD:C_0603_1608Metric, F.Cu at (140.4, 94.2)
- added C9: 600S180FT250XT, Capacitor_SMD:C_0603_1608Metric, F.Cu at (140.4, 85.3)
- added L1: MHQ0402PSA2N9ST000, Inductor 2.9 nH:Untitled, F.Cu at (140.5, 87.2)
- added L2: MHQ0402PSA2N9ST000, Inductor 2.9 nH:Untitled, F.Cu at (140.5, 99.2)
- added R3: RC0603JR-070RL, Resistor_SMD:R_0603_1608Metric, F.Cu at (159.8, 100.2)
- added R4: RC0603FR-0710KL, Resistor_SMD:R_0603_1608Metric, F.Cu at (175.8, 101.5)
- added R5: RC0603FR-0710KL, Resistor_SMD:R_0603_1608Metric, F.Cu at (169.6, 98.3)
- added R6: RC0603FR-0710KL, Resistor_SMD:R_0603_1608Metric, F.Cu at (175.8, 98.4)
- added TeamNames2: ~, Team_Names:Untitled, F.Cu at (160.1, 44.0)
- added U18: DAC6551AQDGKRQ1, DAC6551AQDGKRQ1:DGK8_TEX, F.Cu at (164.8, 99.8)
- added U19: OPA1612AIDRGT, OPA1612AIDRGT:DRG8_1P2X2P0_TEX, F.Cu at (172.7, 99.2)
- added U20: ~, Resistor_SMD:R_0603_1608Metric, F.Cu at (142.8, 83.5)
- added U21: ~, Resistor_SMD:R_0603_1608Metric, F.Cu at (142.8, 96.0)
- C11, C12: value GRM1885C1H431JA01D -> 600S1R8BT250XT
- L3: footprint Inductor 4.7uH:IND_LQM18PxxxxFRx_MUR-M -> Inductor 3.3 uH:INDC1608X95N
- U16: value LDO40LPU33RY -> LDO40LPU55RY
- moved C11 32.2 mm to (142.8, 87.0), turned to 0 degrees
- moved C12 28.8 mm to (142.8, 99.0), turned to 0 degrees
- moved CR1 8.33 mm to (144.6, 77.5)
- moved CR2 7.15 mm to (147.6, 70.8), turned to 180 degrees
- moved C13 5.98 mm to (164.7, 104.2), turned to 0 degrees
- moved R2 4.81 mm to (163.9, 97.0)
- moved C14 4.68 mm to (164.8, 102.6), turned to 0 degrees
- moved C1 3.23 mm to (159.9, 60.5)
- moved C2 3.23 mm to (159.1, 69.0)
- moved C27 3.23 mm to (152.3, 59.4)
- moved C28 3.23 mm to (152.5, 66.3)
- moved R13 3.23 mm to (161.0, 69.0)
- moved R14 3.23 mm to (158.3, 66.4)
- moved U16 3.23 mm to (156.7, 61.2)
- moved U17 3.23 mm to (155.9, 69.3)
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Connections:
- C11 pad 1: Net-(U5-IN+) -> Net-(C11-Pad1)
- C11 pad 2: Net-(IC3-AIN0) -> GND
- C12 pad 1: Net-(U5-IN-) -> Net-(C10-Pad2)
- C12 pad 2: Net-(IC3-AIN1) -> GND
- C19 pad 2: +5V -> Net-(U9-5V)
- C20 pad 2: +5V -> Net-(U9-5V)
- C27 pad 2: Net-(U16-EN) -> +6V
- C28 pad 2: Net-(U17-EN) -> +6V
- CR1 pad 2: Net-(U17-EN) -> +6V
- CR2 pad 1: /V_Source2 -> +6V
- CR2 pad 2: Net-(U16-EN) -> Net-(U9-5V)
- InvertedF0 pad 1: /RF0 -> Net-(InvertedF0-RF)
- InvertedF1 pad 1: /RF1 -> Net-(InvertedF1-RF)
- R2 pad 1: /QPG_TX -> /Data -
- R2 pad 2: /DAC_SDA -> /SCLK
- U16 pad 2: Net-(U16-EN) -> +6V
- U16 pad 3: Net-(U16-EN) -> +6V
- U17 pad 2: Net-(U17-EN) -> +6V
- U17 pad 3: Net-(U17-EN) -> +6V
- U17 pad 5: Net-(U17-ADJ) -> +3.3V
- U17 pad 6: Net-(U17-ADJ) -> unconnected-(U17-ADJ-Pad6)
- U3 pad 17: /DAC_SCL -> /SYNC
- U3 pad 21: /ALERT/RDY -> unconnected-(U3-GPIO5_(PROG_ENN)-Pad21)
- U5 pad A1: Net-(U5-IN+) -> /OUTA
- U5 pad C1: Net-(U5-IN-) -> /OUTB
- U9 pad 1: +5V -> Net-(U9-5V)
Routing:
- net /GNDRF1: track 61.1 -> 0.02 mm
- net /GNDRF0: track 51.5 -> 0.00 mm
- net +6V: track 0.00 -> 44.1 mm, vias 0 -> 3
- net Net-(U9-5V): track 0.00 -> 41.2 mm, vias 0 -> 2
- net +5V: track 180.1 -> 156.4 mm
- net /ALERT/RDY: track 23.6 -> 0.00 mm, vias 2 -> 0
- net Net-(U5-IN+): track 21.6 -> 0.00 mm
- net /OUTA: track 0.00 -> 20.5 mm
- net /DAC_OUT: track 0.00 -> 19.7 mm
- net /V_Source2: track 55.3 -> 39.0 mm, vias 2 -> 1
- net /DAC_SCL: track 12.9 -> 0.00 mm
- net /RF0: track 28.0 -> 15.3 mm, vias 0 -> 2
- net /OUTB: track 0.00 -> 9.76 mm
- net Net-(InvertedF1-RF): track 0.00 -> 7.90 mm
- net Net-(U16-EN): track 7.56 -> 0.00 mm
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- added copper zone on In3.Cu, net (none)
- added copper zone on In2.Cu, net GND
- added copper zone on In3.Cu, net GND

Commit message: Add files via upload
Parts:
- removed C19: CL10B105KP8NNNC, Capacitor_SMD:C_0603_1608Metric
- removed C20: CL10B104JB8NNNC, Capacitor_SMD:C_0603_1608Metric
- removed CR2: CMS11TE12L_Q_M, Diode CMS11:M-FLAT_TOS-M
- removed R13: RC0603JR-076K8L, Resistor_SMD:R_0603_1608Metric
- removed R14, R5: RC0603FR-0710KL, Resistor_SMD:R_0603_1608Metric
- removed R2: RC0603JR-070RL, Resistor_SMD:R_0603_1608Metric
- removed U1, U11, U2, U6, U7, U8: ~, Resistor_SMD:R_0603_1608Metric
- removed U9: ~, AU-Y1005:LED Header
- added C33: DNP, Capacitor_SMD:C_0603_1608Metric, F.Cu at (153.5, 102.3)
- added C34: DNP, Capacitor_SMD:C_0603_1608Metric, F.Cu at (157.8, 103.6)
- added C35: CL10A225KO8NNNC, Capacitor_SMD:C_0603_1608Metric, F.Cu at (149.6, 90.9)
- added C36: CL10A475KP8NNNC, Capacitor_SMD:C_0603_1608Metric, F.Cu at (149.6, 89.3)
- added C37: DNP, Capacitor_SMD:C_0603_1608Metric, F.Cu at (172.8, 82.5)
- added C38: DNP, Capacitor_SMD:C_0603_1608Metric, F.Cu at (172.8, 80.9)
- added C39: DNP, Capacitor_SMD:C_0603_1608Metric, F.Cu at (165.7, 78.8)
- added C40: DNP, Capacitor_SMD:C_0603_1608Metric, F.Cu at (165.7, 77.1)
- added J10: 901200121, Test_Header_1POS:CONN_SD-90120-001_01_MOL, F.Cu at (176.0, 87.4)
- added J11: 901200121, Test_Header_1POS:CONN_SD-90120-001_01_MOL, F.Cu at (175.5, 77.5)
- added J12: 901200121, Test_Header_1POS:CONN_SD-90120-001_01_MOL, F.Cu at (168.6, 72.6)
- added J13: 901200121, Test_Header_1POS:CONN_SD-90120-001_01_MOL, F.Cu at (154.3, 86.4)
- added J14: 901200121, Test_Header_1POS:CONN_SD-90120-001_01_MOL, F.Cu at (149.5, 86.3)
- added J15: 901200121, Test_Header_1POS:CONN_SD-90120-001_01_MOL, F.Cu at (168.7, 108.9)
- added J16: 901200121, Test_Header_1POS:CONN_SD-90120-001_01_MOL, F.Cu at (155.3, 108.2)
- added J18: 901200121, Test_Header_1POS:CONN_SD-90120-001_01_MOL, F.Cu at (163.7, 86.0)
- added J2: 901200121, Test_Header_1POS:CONN_SD-90120-001_01_MOL, F.Cu at (166.2, 95.6)
- added J6: 901200121, Test_Header_1POS:CONN_SD-90120-001_01_MOL, F.Cu at (145.2, 106.6)
- added J7: 901200121, Test_Header_1POS:CONN_SD-90120-001_01_MOL, F.Cu at (176.4, 94.1)
- added J8: 901200121, Test_Header_1POS:CONN_SD-90120-001_01_MOL, F.Cu at (191.8, 94.5)
- added J9: 901200121, Test_Header_1POS:CONN_SD-90120-001_01_MOL, F.Cu at (192.5, 85.8)
- C16, C4: value CL10A106KP8NNNC -> CL10B105KP8NNNC
- U20, U21: value ~ -> DNP
- moved C24 14.5 mm to (155.5, 73.9), turned to 180 degrees
- moved C23 11.4 mm to (155.5, 75.5), turned to 180 degrees
- moved R12 5.26 mm to (163.2, 78.0)
- moved C32 5.02 mm to (145.0, 100.0), turned to 0 degrees
- moved C30 4.51 mm to (144.4, 84.4), turned to 90 degrees
- moved C31 4.21 mm to (144.4, 88.4)
- moved C11 3.63 mm to (141.0, 83.9), turned to 90 degrees
- moved C29 3.52 mm to (142.6, 97.1), turned to 90 degrees
- moved J4 3.13 mm to (172.0, 75.0)
- moved L1 3.04 mm to (143.4, 86.4), turned to 0 degrees
- moved C12 2.65 mm to (141.0, 97.1), turned to 90 degrees
- moved U20 2.57 mm to (141.7, 81.2)
- moved C9 1.79 mm to (139.3, 83.9)
- moved C7 1.79 mm to (139.3, 80.5)
- moved L2 1.72 mm to (142.1, 100.0), turned to 0 degrees
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Connections:
- InvertedF0 pad 1: Net-(InvertedF0-RF) -> /GNDRF0
- InvertedF0 pad 2: /GNDRF0 -> Net-(InvertedF0-RF)
- InvertedF1 pad 1: Net-(InvertedF1-RF) -> /GNDRF1
- InvertedF1 pad 2: /GNDRF1 -> Net-(InvertedF1-RF)
- U19 pad 2: Net-(U19--INA) -> /OUTA
- U3 pad 13: /X32MP -> /X32MP_CRYSTAL
- U3 pad 14: /X32MN -> /X32MN_CRYSTAL
- U3 pad 18: /Data + -> unconnected-(U3-GPIO2_(USBP)-Pad18)
- U3 pad 19: /Data - -> /SCLK
- Y1 pad 1: /X32MN -> /X32MP_CRYSTAL
- Y1 pad 3: /X32MP -> /X32MN_CRYSTAL
Routing:
- net /Data +: track 60.7 -> 0.00 mm, vias 1 -> 0
- net Net-(U9-5V): track 41.2 -> 0.00 mm, vias 2 -> 0
- net /Data -: track 28.2 -> 0.00 mm, vias 2 -> 0
- net Net-(InvertedF1-RF): track 7.90 -> 27.4 mm
- net Net-(InvertedF0-RF): track 7.37 -> 20.1 mm
- net /RF1: track 18.5 -> 8.96 mm, vias 2 -> 0
- net GND: track 107.2 -> 115.5 mm, vias 18 -> 17
- net /QPG_RX: track 17.6 -> 25.0 mm
- net /X32MN_CRYSTAL: track 0.00 -> 7.27 mm
- net Net-(U5-VO-): track 16.2 -> 23.1 mm
- net /SCLK: track 4.05 -> 10.5 mm
- net /X32MN: track 6.20 -> 0.00 mm, vias 2 -> 0
- net /X32MP_CRYSTAL: track 0.00 -> 6.06 mm
- net /OUTA: track 20.5 -> 24.9 mm
- net +6V: track 44.1 -> 39.8 mm
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- added copper zone on B.Cu, net GND
- added copper zone on F.Cu, net GND
- removed copper zone on F.Cu, net (none)
- removed copper zone on In3.Cu, net (none)

Commit message: Add files via upload
Parts:
- removed J15, J16, J18: 901200121, Test_Header_1POS:CONN_SD-90120-001_01_MOL
- removed R3: RC0603JR-070RL, Resistor_SMD:R_0603_1608Metric
- removed R4, R6: RC0603FR-0710KL, Resistor_SMD:R_0603_1608Metric
- removed U19: OPA1612AIDRGT, OPA1612AIDRGT:DRG8_1P2X2P0_TEX
- C3: value CL10B104JB8NNNC -> CL10B105KP8NNNC
- J10, J11, J12, J13, J14, J2, J6, J7, J8, J9: value 901200121 -> 22032021; footprint Test_Header_1POS:CONN_SD-90120-001_01_MOL -> Speaker Header:CONN_SD-4030-0001_02_MOL
- moved J8 43.2 mm to (149.8, 84.5), turned to 90 degrees
- moved J13 25.4 mm to (167.9, 107.9), turned to 0 degrees
- moved J14 22.0 mm to (152.8, 108.0), turned to 0 degrees
- moved J7 21.1 mm to (156.7, 86.5), turned to 180 degrees
- moved J9 16.7 mm to (175.9, 87.1), turned to 90 degrees
- moved C4 15.9 mm to (169.5, 88.1)
- moved J10 12.2 mm to (163.8, 86.3), turned to 0 degrees
- moved J11 11.2 mm to (165.9, 83.3), turned to 180 degrees
- moved J12 6.94 mm to (175.1, 75.0), turned to -90 degrees
- moved J2 6.29 mm to (171.5, 99.0)
- moved C3 5.90 mm to (171.2, 96.5)
- moved J6 1.42 mm to (145.5, 108.0)
- moved C27 0.09 mm to (152.3, 59.3)
Connections:
- net /SCLK renamed /DAC_SCLK
- net /SHUTDOWN renamed /AUDIO_AMP_SHUTDOWN
- net /SYNC renamed /DAC_SYNC
- C3 pad 1: GND -> /DAC_OUT
- C3 pad 2: +3.3V -> Net-(U5-IN-)
- C4 pad 2: +3.3V -> Net-(U5-IN+)
- J13 pad 1: /DATA -> /ULT_SEN_QPG_TX
- J14 pad 1: /CLOCK -> /ULT_SEN_QPG_RX
- J3 pad 2: /QPG_RX -> /ULT_SEN_QPG_RX
- J3 pad 3: /QPG_TX -> /ULT_SEN_QPG_TX
- J7 pad 1: /OUTB -> /MIC_DATA
- J8 pad 1: Net-(U19--INB) -> /MIC_CLOCK
- U18 pad 7: /MOSI -> /DAC_MOSI
- U3 pad 12: unconnected-(U3-ANIO1_GPIO29-Pad12) -> /DAC_MOSI
- U3 pad 15: /QPG_RX -> /ULT_SEN_QPG_RX
- U3 pad 16: /QPG_TX -> /ULT_SEN_QPG_TX
- U3 pad 28: /DATA -> /MIC_DATA
- U3 pad 29: /CLOCK -> /MIC_CLOCK
- U4 pad 3: /DATA -> /MIC_DATA
- U4 pad 4: /CLOCK -> /MIC_CLOCK
- U5 pad A1: /OUTA -> Net-(U5-IN+)
- U5 pad C1: /OUTB -> Net-(U5-IN-)
Routing:
- net /ULT_SEN_QPG_RX: track 0.00 -> 27.3 mm, vias 0 -> 1
- net /QPG_RX: track 25.0 -> 0.00 mm, vias 1 -> 0
- net /OUTA: track 24.9 -> 0.00 mm
- net /ULT_SEN_QPG_TX: track 0.00 -> 21.1 mm, vias 0 -> 1
- net /QPG_TX: track 19.1 -> 0.00 mm, vias 1 -> 0
- net /OUTB: track 14.0 -> 0.00 mm
- net /MIC_CLOCK: track 0.00 -> 13.7 mm, vias 0 -> 2
- net /DAC_OUT: track 22.3 -> 8.97 mm
- net /CLOCK: track 12.1 -> 0.00 mm, vias 2 -> 0
- net /DAC_MOSI: track 0.00 -> 10.7 mm, vias 0 -> 2
- net /MIC_DATA: track 0.00 -> 10.4 mm, vias 0 -> 2
- net /DATA: track 10.1 -> 0.00 mm, vias 2 -> 0
- net GND: track 115.5 -> 108.1 mm, vias 17 -> 24
- net Net-(U5-VO-): track 23.1 -> 29.1 mm
- net +3.3V: track 46.6 -> 42.0 mm, vias 10 -> 8
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
Commit message: Add files via upload
Parts:
- removed InvertedF0: ~, Antenna:InvertedF
- added J15: SMA-J-P-H-ST-TH1, SMA_50Ohm_FEMALE:CONN_SMA-J-P-H-ST-TH1_SAI, F.Cu at (122.7, 85.5)
- moved C7 16.9 mm to (126.0, 91.0), turned to 180 degrees
- moved U20 16.1 mm to (128.4, 90.2), turned to 90 degrees
- moved C9 11.3 mm to (130.6, 91.0), turned to 0 degrees
- moved L1 10.5 mm to (134.0, 91.0)
- moved C11 10.4 mm to (132.8, 90.3)
- moved C30 10.3 mm to (136.0, 90.3)
- moved C21 6.92 mm to (140.8, 107.7)
- moved C22 6.92 mm to (140.8, 109.4)
- moved U10 6.92 mm to (138.3, 111.9)
- moved C31 6.72 mm to (138.2, 91.0), turned to 0 degrees
- moved C29 5.46 mm to (146.1, 101.3), turned to -90 degrees
- moved C12 4.62 mm to (142.8, 101.3), turned to -90 degrees
- moved C10 3.36 mm to (141.3, 99.8)
- moved C32 3.32 mm to (148.3, 100.6)
- moved U21 3.15 mm to (140.4, 97.6), turned to 180 degrees
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Connections:
- net +3.3V renamed /3.3V
- net +5V renamed /5V
- net +6V renamed /6V
- C10 pad 1: Net-(C10-Pad1) -> /RF1+
- C10 pad 2: Net-(C10-Pad2) -> /RF1+
- C11 pad 1: Net-(C11-Pad1) -> /RF0+
- C11 pad 2: GND -> /RF0-
- C12 pad 1: Net-(C10-Pad2) -> /RF1+
- C12 pad 2: GND -> /RF1-
- C29 pad 1: Net-(C29-Pad1) -> /RF1+
- C29 pad 2: GND -> /RF1-
- C30 pad 2: GND -> /RF0-
- C31 pad 2: /RF0 -> /RF0+
- C32 pad 1: Net-(C29-Pad1) -> /RF1+
- C32 pad 2: /RF1 -> /RF1+
- C7 pad 1: Net-(InvertedF0-RF) -> /RF0+
- C7 pad 2: Net-(C7-Pad2) -> /RF0+
- C8 pad 1: Net-(InvertedF1-RF) -> /RF1+
- C8 pad 2: Net-(C10-Pad1) -> /RF1+
- C9 pad 1: Net-(C7-Pad2) -> /RF0+
- C9 pad 2: Net-(C11-Pad1) -> /RF0+
- InvertedF1 pad 1: /GNDRF1 -> /RF1-
- InvertedF1 pad 2: Net-(InvertedF1-RF) -> /RF1+
- L1 pad 1: Net-(C11-Pad1) -> /RF0+
- L2 pad 1: Net-(C10-Pad2) -> /RF1+
- L2 pad 2: Net-(C29-Pad1) -> /RF1+
- U20 pad 1: Net-(C7-Pad2) -> /RF0+
- U20 pad 2: GND -> /RF0-
- U21 pad 1: Net-(C10-Pad1) -> /RF1+
- U21 pad 2: GND -> /RF1-
- U3 pad 10: /GNDRF1 -> /RF1-
- U3 pad 7: /GNDRF0 -> /RF0-
- U3 pad 8: /RF0 -> /RF0+
- U3 pad 9: /RF1 -> /RF1+
Routing:
- net /RF0-: track 0.00 -> 58.3 mm
- net /RF0+: track 0.00 -> 55.7 mm
- net /RF1-: track 0.00 -> 38.5 mm
- net /RF1+: track 0.00 -> 32.3 mm
- net Net-(InvertedF1-RF): track 27.4 -> 0.00 mm
- net Net-(InvertedF0-RF): track 20.1 -> 0.00 mm
- net /RF0: track 17.5 -> 0.00 mm
- net /RF1: track 8.96 -> 0.00 mm
- net /DB_GPIO: track 38.6 -> 32.6 mm
- net Net-(C11-Pad1): track 5.40 -> 0.00 mm
- net Net-(C10-Pad2): track 4.89 -> 0.00 mm
- net Net-(C29-Pad1): track 3.56 -> 0.00 mm
- net Net-(C7-Pad2): track 3.46 -> 0.00 mm
- net Net-(C10-Pad1): track 3.18 -> 0.00 mm
- net /GNDRF1: track 0.62 -> 0.00 mm
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
Commit message: Add files via upload
Parts:
- moved C8 14.8 mm to (126.7, 98.3), turned to 180 degrees
- moved InvertedF1 14.3 mm to (114.1, 106.3), turned to 0 degrees
- moved C7 12.8 mm to (131.1, 79.3), turned to 90 degrees
- moved U21 11.6 mm to (128.9, 99.2), turned to -90 degrees
- moved C10 10.2 mm to (131.2, 98.3), turned to 0 degrees
- moved C12 9.65 mm to (133.4, 99.1)
- moved L2 9.57 mm to (134.7, 98.3)
- moved C32 9.51 mm to (139.1, 98.3)
- moved C29 9.49 mm to (136.8, 99.1)
- moved U20 9.34 mm to (131.9, 81.6), turned to 0 degrees
- moved C9 7.23 mm to (131.1, 83.8), turned to -90 degrees
- moved C31 7.08 mm to (131.1, 91.4), turned to -90 degrees
- moved L1 4.78 mm to (131.1, 87.2), turned to -90 degrees
- moved J15 4.49 mm to (122.6, 81.1)
- moved C11 4.34 mm to (131.9, 86.0), turned to 0 degrees
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Connections:
- C11 pad 2: /RF0- -> GND
- C12 pad 2: /RF1- -> GND
- C29 pad 2: /RF1- -> GND
- C30 pad 2: /RF0- -> GND
- InvertedF1 pad 1: /RF1- -> GND
- U20 pad 2: /RF0- -> GND
- U21 pad 2: /RF1- -> GND
- U3 pad 10: /RF1- -> GND
- U3 pad 7: /RF0- -> GND
Routing:
- net /RF0-: track 58.3 -> 0.00 mm
- net /RF1-: track 38.5 -> 0.00 mm
- net /RF0+: track 55.7 -> 41.6 mm
- net /3.3V: track 42.0 -> 36.1 mm
- net /RF1+: track 32.3 -> 28.3 mm
- net GND: track 108.1 -> 111.4 mm, vias 20 -> 263
- net Net-(U3-VDDANA): track 4.68 -> 7.80 mm
- net Net-(U3-LXL_GPIO20): track 5.07 -> 7.89 mm
- net Net-(U3-VDDCORE): track 6.65 -> 9.41 mm
- net /DB_GPIO: track 32.6 -> 30.7 mm
- net Net-(U3-LXH_GPIO19): track 6.72 -> 5.53 mm
- net /V_Source1: track 32.0 -> 31.2 mm
- net /DAC_MOSI: track 10.7 -> 11.2 mm

Commit message: Add files via upload
Parts:
- moved C8 0.05 mm to (126.7, 98.3), turned to 0 degrees
- turned C7 to -90 degrees
Connections:
- C10 pad 1: /RF1+ -> Net-(C10-Pad1)
- C10 pad 2: /RF1+ -> Net-(C10-Pad2)
- C11 pad 1: /RF0+ -> Net-(C11-Pad1)
- C12 pad 1: /RF1+ -> Net-(C10-Pad2)
- C29 pad 1: /RF1+ -> Net-(C29-Pad1)
- C32 pad 1: /RF1+ -> Net-(C29-Pad1)
- C7 pad 1: /RF0+ -> Net-(C7-Pad1)
- C7 pad 2: /RF0+ -> Net-(C7-Pad2)
- C8 pad 1: /RF1+ -> Net-(InvertedF1-RF)
- C8 pad 2: /RF1+ -> Net-(C10-Pad1)
- C9 pad 1: /RF0+ -> Net-(C7-Pad2)
- C9 pad 2: /RF0+ -> Net-(C11-Pad1)
- InvertedF1 pad 2: /RF1+ -> Net-(InvertedF1-RF)
- J15 pad 1: /RF0+ -> Net-(C7-Pad1)
- L1 pad 1: /RF0+ -> Net-(C11-Pad1)
- L2 pad 1: /RF1+ -> Net-(C10-Pad2)
- L2 pad 2: /RF1+ -> Net-(C29-Pad1)
- U20 pad 1: /RF0+ -> Net-(C7-Pad2)
- U21 pad 1: /RF1+ -> Net-(C10-Pad1)
Routing:
- net GND: track 111.4 -> 94.0 mm, vias 263 -> 276
- net /RF0+: track 41.6 -> 24.9 mm
- net Net-(C7-Pad1): track 0.00 -> 11.1 mm
- net /RF1+: track 28.3 -> 17.8 mm
- net /3.3V: track 36.1 -> 40.9 mm
- net Net-(C7-Pad2): track 0.00 -> 3.11 mm
- net Net-(C10-Pad1): track 0.00 -> 3.02 mm
- net Net-(C10-Pad2): track 0.00 -> 2.75 mm
- net Net-(C11-Pad1): track 0.00 -> 2.66 mm
- net Net-(C29-Pad1): track 0.00 -> 2.65 mm
- net Net-(InvertedF1-RF): track 0.00 -> 2.27 mm
