File: Electrical/Hardware/Schematics/QORVO_RADIO2.kicad_sch (KiCad schematic)
At the start: 62 parts, among them IC3 ADS1114BQDGSRQ1, J2 3220-10-0100-00, J3 22032041, J4 22032021, J5 22032041, SW1 OS102011MS2QN1, U10 22032021, U16 LDO40LPU33RY, U17 LDO40LPU33RY, Y1 8Q-32.000MEEV-T

Commit message: Add files via upload
Parts:
- removed J2: 3220-10-0100-00, J-Link Header:CONN_3220-10-0100-00_CNC, symbol J-Link Header:3220-10-0100-00
- added J1: GRPB052VWQS-RC, GRPB052VWQS-RC:CONN_GRPB052_SUL, symbol GRPB052VWQS-RC:GRPB052VWQS-RC
Connections:
- net +3.3V: now also J1.1 (VTref)
- net GND: now also U16.7 (EPAD), U17.7 (EPAD), J1.3 (GND), J1.5 (GND)
- net JTAG_TCK: now also J1.4 (TCK)
- net JTAG_TDI: now also J1.8 (TDI)
- net JTAG_TDO: now also J1.6 (TDO)
- net JTAG_TMS: now also J1.2 (TMS)
- net JTAG_nRESET: now also J1.10 (nRESET)
Changed lines of the file:
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@@
 	(wire
 		(pts
+			(xy 237.49 107.95) (xy 237.49 114.3)
+		)
+		(stroke
+			(width 0)
+			(type default)
+		)
+	)
+	(wire
+		(pts
 			(xy 213.36 176.53) (xy 199.39 176.53)
 		)
@@
 	(wire
 		(pts
+			(xy 232.41 24.13) (xy 232.41 26.67)
+		)
+		(stroke
+			(width 0)
+			(type default)
+		)
+	)
+	(wire
+		(pts
 			(xy 499.11 332.74) (xy 499.11 334.01)
 		)
@@
 	(wire
 		(pts
+			(xy 233.68 114.3) (xy 237.49 114.3)
+		)
+		(stroke
+			(width 0)
+			(type default)
+		)
+	)
+	(wire
+		(pts
 			(xy 485.14 237.49) (xy 485.14 246.38)
 		)
@@
 	(wire
 		(pts
+			(xy 226.06 26.67) (xy 232.41 26.67)
+		)
+		(stroke
+			(width 0)
+			(type default)
+		)
+	)
+	(wire
+		(pts
 			(xy 77.47 326.39) (xy 81.28 326.39)
 		)
@@
 	)
 	(symbol
-		(lib_id "J-Link Header:3220-10-0100-00")
-		(at 480.06 54.61 0)
-		(unit 1)
-		(exclude_from_sim no)
-		(in_bom yes)
-		(on_board yes)
-		(dnp no)
-		(fields_autoplaced yes)
-		(property "Reference" "J2"
-			(at 494.03 64.7699 0)
-			(effects
-				(font
-					(size 1.524 1.524)
-				)
-				(justify left)
-			)
-		)
-		(property "Value" "3220-10-0100-00"
-			(at 494.03 67.3099 0)
-			(effects
-				(font
-					(size 1.524 1.524)
-				)
-				(justify left)
-			)
-		)
-		(property "Footprint" "J-Link Header:CONN_3220-10-0100-00_CNC"
-			(at 480.06 54.61 0)
-			(effects
-				(font
-					(size 1.27 1.27)
-					(italic yes)
-				)
-				(hide yes)
-			)
-		)
-		(property "Datasheet" "3220-10-0100-00"
-			(at 480.06 54.61 0)
-			(effects
-				(font
-					(size 1.27 1.27)
-					(italic yes)
-				)
-				(hide yes)
-			)
-		)
-		(property "Description" ""
-			(at 480.06 54.61 0)
-			(effects
-				(font
-					(size 1.27 1.27)
-				)
-				(hide yes)
-			)
-		)
-		(pin "6"
-		)
-		(pin "3"
-		)
-		(pin "7"
-		)
-		(pin "10"
-		)
-		(pin "5"
-		)
-		(pin "4"
-		)
-		(pin "1"
-		)
-		(pin "9"
-		)
-		(pin "2"
-		)
-		(pin "8"
-		)
-		(instances
-			(project ""
-				(path "/857d4a07-0150-4c4b-a0bc-a2b2a01a1105"
-					(reference "J2")
-					(unit 1)
-				)
-			)
-		)
-	)
-	(symbol
 		(lib_id "Capacitor 1 uF:CL10B105KP8NNNC")
 		(at 213.36 189.23 0)
@@
 		(property "Footprint" "AU-Y1005:LED Header"
 			(at 504.19 325.12 0)
+			(show_name yes)
 			(effects
 				(font
@@
 	)
 	(symbol
+		(lib_id "power:GND")
+		(at 237.49 107.95 180)
+		(unit 1)
+		(exclude_from_sim no)
+		(in_bom yes)
+		(on_board yes)
+		(dnp no)
+		(fields_autoplaced yes)
+		(property "Reference" "#PWR09"
+			(at 237.49 101.6 0)
+			(effects
+				(font
+					(size 1.27 1.27)
+				)
+				(hide yes)
+			)
+		)
+		(property "Value" "GND"
+			(at 237.49 102.87 0)
+			(effects
+				(font
+					(size 1.27 1.27)
+				)
+			)
+		)
+		(property "Footprint" ""
+			(at 237.49 107.95 0)
+			(effects
+				(font
+					(size 1.27 1.27)
+				)
+				(hide yes)
+			)
+		)
+		(property "Datasheet" ""
+			(at 237.49 107.95 0)
+			(effects
+				(font
+					(size 1.27 1.27)
+				)
+				(hide yes)
+			)
+		)
+		(property "Description" "Power symbol creates a global label with name \"GND\" , ground"
+			(at 237.49 107.95 0)
+			(effects
+				(font
+					(size 1.27 1.27)
+				)
+				(hide yes)
+			)
+		)
+		(pin "1"
+		)
+		(instances
+			(project ""
+				(path "/857d4a07-0150-4c4b-a0bc-a2b2a01a1105"
+					(reference "#PWR09")
+					(unit 1)
+				)
+			)
+		)
+	)
+	(symbol
 		(lib_id "Resistor 1KOhm:RMCF0603FG1K00")
 		(at 278.13 274.32 270)
@@
 	)
 	(symbol
+		(lib_id "GRPB052VWQS-RC:GRPB052VWQS-RC")
+		(at 480.06 54.61 0)
+		(unit 1)
+		(exclude_from_sim no)
+		(in_bom yes)
+		(on_board yes)
+		(dnp no)
+		(fields_autoplaced yes)
+		(property "Reference" "J1"
+			(at 494.03 64.7699 0)
+			(effects
+				(font
+					(size 1.524 1.524)
+				)
+				(justify left)
+			)
+		)
+		(property "Value" "GRPB052VWQS-RC"
+			(at 494.03 67.3099 0)
+			(effects
+				(font
+					(size 1.524 1.524)
+				)
+				(justify left)
+			)
+		)
+		(property "Footprint" "GRPB052VWQS-RC:CONN_GRPB052_SUL"
+			(at 480.06 54.61 0)
+			(effects
+				(font
+					(size 1.27 1.27)
+					(italic yes)
+				)
+				(hide yes)
+			)
+		)
+		(property "Datasheet" "GRPB052VWQS-RC"
+			(at 480.06 54.61 0)
+			(effects
+				(font
+					(size 1.27 1.27)
+					(italic yes)
+				)
+				(hide yes)
+			)
+		)
+		(property "Description" ""
+			(at 480.06 54.61 0)
+			(effects
+				(font
+					(size 1.27 1.27)
+				)
+				(hide yes)
+			)
+		)
+		(pin "8"
+		)
+		(pin "4"
+		)
+		(pin "5"
+		)
+		(pin "7"
+		)
+		(pin "6"
+		)
+		(pin "10"
+		)
+		(pin "1"
+		)
+		(pin "2"
+		)
+		(pin "3"
+		)
+		(pin "9"
+		)
+		(instances
+			(project ""
+				(path "/857d4a07-0150-4c4b-a0bc-a2b2a01a1105"
+					(reference "J1")
+					(unit 1)
+				)
+			)
+		)
+	)
+	(symbol
 		(lib_id "Resistor 0 Ohm:Shunt")
 		(at 332.74 397.51 270)
@@
 					(unit 1)
 				)
+			)
+		)
+	)
+	(symbol
+		(lib_id "power:GND")
+		(at 232.41 24.13 180)
+		(unit 1)
+		(exclude_from_sim no)
+		(in_bom yes)
+		(on_board yes)
+		(dnp no)
+		(fields_autoplaced yes)
+		(property "Reference" "#PWR08"
+			(at 232.41 17.78 0)
+			(effects
+				(font
+					(size 1.27 1.27)
+				)
+				(hide yes)
+			)
+		)
+		(property "Value" "GND"
+			(at 232.41 19.05 0)
+			(effects
+				(font
+					(size 1.27 1.27)
+				)
+			)
+		)
+		(property "Footprint" ""
+			(at 232.41 24.13 0)
+			(effects
+				(font
+					(size 1.27 1.27)
+				)
+				(hide yes)
+			)
+		)
+		(property "Datasheet" ""
+			(at 232.41 24.13 0)
+			(effects
+				(font
+					(size 1.27 1.27)
+				)
+				(hide yes)
+			)
+		)
+		(property "Description" "Power symbol creates a global label with name \"GND\" , ground"
+			(at 232.41 24.13 0)
+			(effects
+				(font
+					(size 1.27 1.27)
+				)
+				(hide yes)
+			)
+		)
+		(pin "1"
+		)
+		(instances
+			(project ""
+				(path "/857d4a07-0150-4c4b-a0bc-a2b2a01a1105"
+					(reference "#PWR08")
+					(unit 1)
+				)

Commit message: Add files via upload
Parts:
- removed C11, C12: GRM1885C1H431JA01D, Capacitor_SMD:C_0603_1608Metric, symbol Capacitor 430pF:GRM1885C1H431JA01D
- removed IC3: ADS1114BQDGSRQ1, ADS1114BQDGSRQ1:SOP50P490X110-10N, symbol ADS1114BQDGSRQ1:ADS1114BQDGSRQ1
- removed R11, R8, R9: RMCF0603FG1K00, Resistor_SMD:R_0603_1608Metric, symbol Resistor 1KOhm:RMCF0603FG1K00
- removed R13: RC0603JR-076K8L, Resistor_SMD:R_0603_1608Metric, symbol Resistor 6.8 KOhm:RC0603JR-076K8L
- removed R14: RC0603FR-0710KL, Resistor_SMD:R_0603_1608Metric, symbol Resistor 10 KOhm:RC0603FR-0710KL
- added C10, C7, C8, C9: 600S180FT250XT, Capacitor_SMD:C_0603_1608Metric, symbol Capacitor 18 pF:600S180FT250XT
- added C11, C12: 600S1R8BT250XT, Capacitor_SMD:C_0603_1608Metric, symbol Capacitor 1.8 pF:600S1R8BT250XT
- added C29, C30: 600S1R5BT250XT4K, Capacitor_SMD:C_0603_1608Metric, symbol Capacitor 18 pF:600S180FT250XT
- added C3: CL10B104JB8NNNC, Capacitor_SMD:C_0603_1608Metric, symbol Capacitor 0.1uF:CL10B104JB8NNNC
- added C31, C32: 600S2R2AT250XT4K, Capacitor_SMD:C_0603_1608Metric, symbol Capacitor 18 pF:600S180FT250XT
- added C4: CL10B105KP8NNNC, Capacitor_SMD:C_0603_1608Metric, symbol Capacitor 10uF:CL10A106KP8NNNC
- added L1, L2: MHQ0402PSA2N9ST000, Inductor 2.9 nH:Untitled, symbol Inductor 2.9 nH:MHQ0402PSA2N9ST000
- added R3: RC0603JR-070RL, Resistor_SMD:R_0603_1608Metric, symbol Resistor 0 Ohm:RC0603JR-070RL
- added R4, R5, R6: RC0603FR-0710KL, Resistor_SMD:R_0603_1608Metric, symbol Resistor 10 KOhm:RC0603FR-0710KL
- added TeamNames1: ~, symbol Team Names:Team_Names
- added TeamNames2: ~, Team_Names:Untitled, symbol Team Names:Team_Names
- added U18: DAC6551AQDGKRQ1, DAC6551AQDGKRQ1:DGK8_TEX, symbol DAC6551AQDGKRQ1:DAC6551AQDGKRQ1
- added U19: OPA1612AIDRGT, OPA1612AIDRGT:DRG8_1P2X2P0_TEX, symbol OPA1612AIDRGT:OPA1612AIDRGT
- added U20, U21: ~, Resistor_SMD:R_0603_1608Metric, symbol Resistor 0 Ohm:Shunt
- C16: value CL10A106KP8NNNC -> CL10B105KP8NNNC
- L3: footprint Inductor 4.7uH:IND_LQM18PxxxxFRx_MUR-M -> Inductor 3.3 uH:INDC1608X95N
- U16: value LDO40LPU33RY -> LDO40LPU55RY
Connections:
- net +3.3V: now also U17.5 (VSENSE), C3.2, C4.2, U18.1 (VDD), U18.2 (VREF), U19.8 (V+)
- net +5V: no longer C19.2, C20.2, U9.1 (5V)
- net Data -: now also R2.1
- net GND: now also C11.2, C12.2, C29.2, C3.1, C30.2, C4.1, U18.8 (GND), U19.4 (V-), U19.5 (+INB), U19.9 (EPAD), U20.2, U21.2
- net QPG_TX: now also R3.1; no longer R2.1
- net RF0: now also C31.2; no longer InvertedF0.1 (RF)
- net RF1: now also C32.2; no longer InvertedF1.1 (RF)
- net V_Source2: no longer CR2.1
- net at U17.6 (ADJ): no longer U17.5 (VSENSE)
- net +6V: now reaches C28.2, CR1.2, U17.2 (EN), U17.3 (VIN)
- net +6V: now also C27.2, CR2.1, U16.2 (EN), U16.3 (VIN)
- net OUTB: now reaches U5.C1 (IN-)
- net OUTB: now also R6.1, U19.7 (OUTB)
- net OUTA: now reaches U5.A1 (IN+)
- net OUTA: now also R5.1, U19.1 (OUTA)
- net ALERT/RDY: no longer names the net of U3.21 (GPIO5_(PROG_ENN))
- net DAC_SCL renamed SYNC
- net SYNC: now also U18.5 (*SYNC)
- net DAC_SDA renamed SCLK
- net SCLK: now also U18.6 (SCLK)
- new net: C7.1, InvertedF0.1 (RF)
- new net: C7.2, C9.1, U20.1
- new net: R5.2, U19.2 (-INA)
- new net: R4.2, R6.2, U19.6 (-INB)
- new net: C8.1, InvertedF1.1 (RF)
- new net: C11.1, C9.2, L1.1
- new net: C30.1, C31.1, L1.2
- new net: C19.2, C20.2, CR2.2, U9.1 (5V)
- new net: C10.2, C12.1, L2.1
- new net: C10.1, C8.2, U21.1
- new net: C29.1, C32.1, L2.2
- new net DAC_OUT: R4.1, U18.3 (VFB), U18.4 (VOUT), U19.3 (+INA)
- new net MOSI: R3.2, U18.7 (DIN)
Other:
- moved on the sheet: C13, C14, C15, C16, C19, C2, C20, CR1, InvertedF0, InvertedF1, J4, R10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

Commit message: Add files via upload
Parts:
- removed C19: CL10B105KP8NNNC, Capacitor_SMD:C_0603_1608Metric, symbol Capacitor 1 uF:CL10B105KP8NNNC
- removed C20: CL10B104JB8NNNC, Capacitor_SMD:C_0603_1608Metric, symbol Capacitor 0.1uF:CL10B104JB8NNNC
- removed CR2: CMS11TE12L_Q_M, Diode CMS11:M-FLAT_TOS-M, symbol Diode CMS11:CMS11TE12L_Q_M
- removed R2: RC0603JR-070RL, Resistor_SMD:R_0603_1608Metric, symbol Resistor 0 Ohm:RC0603JR-070RL
- removed R5: RC0603FR-0710KL, Resistor_SMD:R_0603_1608Metric, symbol Resistor 10 KOhm:RC0603FR-0710KL
- removed U1, U11, U2, U6, U7, U8: ~, Resistor_SMD:R_0603_1608Metric, symbol Resistor 0 Ohm:Shunt
- removed U9: ~, AU-Y1005:LED Header, symbol AU-Y1005:AU-Y1005
- added C33, C34, C37, C38, C39, C40: DNP, Capacitor_SMD:C_0603_1608Metric, symbol Capacitor 10uF:CL10A106KP8NNNC
- added C35: CL10A225KO8NNNC, Capacitor_SMD:C_0603_1608Metric, symbol Capacitor 10uF:CL10A106KP8NNNC
- added C36: CL10A475KP8NNNC, Capacitor_SMD:C_0603_1608Metric, symbol Capacitor 10uF:CL10A106KP8NNNC
- added J10, J11, J12, J13, J14, J15, J16, J18, J2, J6, J7, J8, J9: 901200121, Test_Header_1POS:CONN_SD-90120-001_01_MOL, symbol Test_Header_1POS:901200121
- U20, U21: value ~ -> DNP; now fitted
Connections:
- net Data - is gone; now on net SCLK: U3.19 (GPIO3_(USBN))
- net CLOCK: now also J14.1
- net DAC_OUT: now also J2.1
- net DATA: now also J13.1
- net DB_GPIO: now also J6.1
- net GND: now also C33.2, C34.2, C35.2, C36.2, C37.2, C38.2, C39.2, C40.2
- net GNDRF0: now also InvertedF0.1 (GND); no longer InvertedF0.2 (GND)
- net GNDRF1: now also InvertedF1.1 (GND); no longer InvertedF1.2 (GND)
- net OUTA: now also U19.2 (-INA), J18.1
- net OUTB: now also J7.1
- net QPG_RX: now also J16.1
- net QPG_TX: now also J15.1
- net at C7.1: now also InvertedF0.2 (RF); no longer InvertedF0.1 (RF)
- net at R4.2, R6.2, U19.6 (-INB): now also J8.1
- net at C8.1: now also InvertedF1.2 (RF); no longer InvertedF1.1 (RF)
- net at U3.31 (VDDCORE): now also C36.1
- net at R12.1, U5.A3 (VO-): now also C39.1, J10.1
- net at J4.1, R12.2: now also C40.1, J12.1
- net at R10.1, U5.C3 (VO+): now also C37.1, J9.1
- net at J4.2, R10.2: now also C38.1, J11.1
- net at U3.32 (VDDANA): now also C35.1
- net Data +: no longer names the net of U3.18 (GPIO2_(USBP))
- net X32MN renamed X32MN_CRYSTAL
- net X32MN_CRYSTAL: now also Y1.3, C34.1; no longer Y1.1
- net X32MP renamed X32MP_CRYSTAL
- net X32MP_CRYSTAL: now also Y1.1, C33.1; no longer Y1.3
Other:
- moved on the sheet: C10, C11, C12, C13, C14, C15, C16, C17, C18, C2, C21, C22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

Commit message: Add files via upload
Parts:
- removed C3: CL10B104JB8NNNC, Capacitor_SMD:C_0603_1608Metric, symbol Capacitor 0.1uF:CL10B104JB8NNNC
- removed C4: CL10B105KP8NNNC, Capacitor_SMD:C_0603_1608Metric, symbol Capacitor 10uF:CL10A106KP8NNNC
- removed J10, J11, J12, J13, J14, J15, J16, J18, J2, J6, J7, J8, J9: 901200121, Test_Header_1POS:CONN_SD-90120-001_01_MOL, symbol Test_Header_1POS:901200121
- removed R3: RC0603JR-070RL, Resistor_SMD:R_0603_1608Metric, symbol Resistor 0 Ohm:RC0603JR-070RL
- removed R4, R6: RC0603FR-0710KL, Resistor_SMD:R_0603_1608Metric, symbol Resistor 10 KOhm:RC0603FR-0710KL
- removed U19: OPA1612AIDRGT, OPA1612AIDRGT:DRG8_1P2X2P0_TEX, symbol OPA1612AIDRGT:OPA1612AIDRGT
- added C3, C4: CL10B105KP8NNNC, Capacitor_SMD:C_0603_1608Metric, symbol Capacitor 1 uF:CL10B105KP8NNNC
- added J10, J11, J12, J13, J14, J2, J6, J7, J8, J9: 22032021, CONN_SD-4030-0001_02_MOL, symbol Speaker header:22032021
Connections:
- net MOSI is gone; now on net DAC_MOSI: U18.7 (DIN)
- net DAC_OUT: now also C3.1, J2.1
- net DB_GPIO: now also J6.1
- net GND: now also C4.1, J10.2, J11.2, J12.2, J13.2, J14.2, J2.2, J6.2, J7.2, J8.2, J9.2
- net at C37.1, R10.1, U5.C3 (VO+): now also J9.1
- net at C38.1, J4.2, R10.2: now also J11.1
- net at C39.1, R12.1, U5.A3 (VO-): now also J10.1
- net at C40.1, J4.1, R12.2: now also J12.1
- net DAC_MOSI: now reaches U3.12 (ANIO1_GPIO29)
- net CLOCK renamed MIC_CLOCK
- net MIC_CLOCK: now also J8.1
- net DATA renamed MIC_DATA
- net MIC_DATA: now also J7.1
- net OUTA: no longer names the net of U5.A1 (IN+)
- net OUTA: now also C4.2
- net OUTB: no longer names the net of U5.C1 (IN-)
- net OUTB: now also C3.2
- net QPG_RX renamed ULT_SEN_QPG_RX
- net ULT_SEN_QPG_RX: now also J14.1
- net QPG_TX renamed ULT_SEN_QPG_TX
- net ULT_SEN_QPG_TX: now also J13.1
- net SCLK renamed DAC_SCLK
- net SHUTDOWN renamed AUDIO_AMP_SHUTDOWN
- net SYNC renamed DAC_SYNC
Other:
- moved on the sheet: C13, C14, C15, C16, C21, C22, C33, C34, C37, C38, C39, C40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

Commit message: Add files via upload
Parts:
- removed InvertedF0: ~, Antenna:InvertedF, symbol Inverted_F_Antenna:_1
- added J15: SMA-J-P-H-ST-TH1, SMA_50Ohm_FEMALE:CONN_SMA-J-P-H-ST-TH1_SAI, symbol SMA_50Ohm_FEMALE:SMA-J-P-H-ST-TH1
- J10, J13, J14, J9: footprint CONN_SD-4030-0001_02_MOL -> Speaker Header:CONN_SD-4030-0001_02_MOL
Connections:
- net RF0 is gone; now on net RF0+: C31.2, U3.8 (RF0)
- net RF1 is gone; now on net RF1+: C32.2, U3.9 (RF1)
- net GND: no longer C11.2, C12.2, C29.2, C30.2, U20.2, U21.2
- net RF0+: now reaches C7.1
- net RF0+: now also C11.1, C7.2, C9.1, C9.2, L1.1, U20.1, J15.1
- net RF1+: now reaches C8.1, InvertedF1.2 (RF)
- net RF1+: now also C10.1, C10.2, C12.1, C29.1, C32.1, C8.2, L2.1, L2.2, U21.1
- net +3.3V renamed 3.3V
- net +5V renamed 5V
- net +6V renamed 6V
- net GNDRF0 renamed RF0-
- net RF0-: now also C11.2, C30.2, U20.2, J15.2 (GND1), J15.3 (GND2), J15.4 (GND3), J15.5 (GND4)
- net GNDRF1 renamed RF1-
- net RF1-: now also C12.2, C29.2, U21.2
Other:
- moved on the sheet: C4

Commit message: Add files via upload
Connections:
- net RF1- is gone; now on net GND: C12.2, C29.2, InvertedF1.1 (GND), U21.2, U3.10 (GNDRF1)
- net GND: now also C11.2, C30.2, J15.0 (GND), U20.2, U3.7 (GNDRF0)
- removed net RF0-: C11.2, C30.2, J15.2 (GND1), J15.3 (GND2), J15.4 (GND3), J15.5 (GND4), U20.2, U3.7 (GNDRF0)

Commit message: Add files via upload
Connections:
- net GND: now also U3.0 (GND3); no longer U3.34 (GND1), U3.35 (GND2), U3.36 (GND3), U3.37 (GND4)
- net RF0+: no longer C11.1, C7.1, C7.2, C9.1, C9.2, J15.1, L1.1, U20.1
- net RF1+: no longer C10.1, C10.2, C12.1, C29.1, C32.1, C8.1, C8.2, InvertedF1.2 (RF), L2.1, L2.2, U21.1
- new net: C7.1, J15.1
- new net: C7.2, C9.1, U20.1
- new net: C8.1, InvertedF1.2 (RF)
- new net: C11.1, C9.2, L1.1
- new net: C10.2, C12.1, L2.1
- new net: C10.1, C8.2, U21.1
- new net: C29.1, C32.1, L2.2
